Commit message: object picking

File: models/urdf/ffw_sg2_rev1_follower/ffw_sg2_follower.urdf (robot description, URDF)
Before this commit: robot ffw_sg2_follower, 40 links, 39 joints
Links:
- added link gripper_l_tcp
- added link gripper_r_tcp
Joints:
- added joint gripper_l_tcp_joint: type fixed, parent gripper_l_rh_p12_rn_base, child gripper_l_tcp, origin xyz=0 0 0.1 rpy=0 0 0
- added joint gripper_r_tcp_joint: type fixed, parent gripper_r_rh_p12_rn_base, child gripper_r_tcp, origin xyz=0 0 0.10 rpy=0 0 0
