Commit message: force_ik

File: models/urdf/common/follower/ffw_follower_body.xacro (robot description, xacro)
@@ -110,5 +110,5 @@
          <parent link="${prefix}arm_base_link" />
          <child link="${prefix}arm_l_link1" />
-         <origin xyz="0 0.1045 0" rpy="0 0 0" />
+         <origin xyz="0 -0.1045 0" rpy="0 0 0" />
          <axis xyz="0 1 0" />
          <limit velocity="4.8" effort="1000" lower="-3.14" upper="3.14" />

File: models/urdf/ffw_sg2_rev1_follower/ffw_sg2_follower.urdf (robot description, URDF)
Before this commit: robot ffw_sg2_follower, 40 links, 39 joints
Joints:
- joint arm_l_joint1: origin xyz=0 0.1045 0 rpy=0 0 0 -> xyz=0 0.1045 0 rpy=0 0.047 0
- joint arm_r_joint1: origin xyz=0 -0.1045 0 rpy=0 0 0 -> xyz=0 -0.1045 0 rpy=0 0.025 0

Commit message: modified joint 7 limit

File: models/urdf/common/follower/ffw_follower_body.xacro (robot description, xacro)
@@ -304,5 +304,5 @@
          <origin xyz="0 0 -0.0885" rpy="0 0 0" />
          <axis xyz="1 0 0" />
-         <limit velocity="4.8" effort="1000" lower="-1.8201" upper="1.5804" />
+         <limit velocity="4.8" effort="1000" lower="-1.9199" upper="1.2217" />
          <dynamics damping="0.1" />
       </joint>
@@ -531,5 +531,5 @@
          <origin xyz="0 0 -0.0885" rpy="0 0 0" />
          <axis xyz="1 0 0" />
-         <limit velocity="4.8" effort="1000" lower="-1.5804" upper="1.8201" />
+         <limit velocity="4.8" effort="1000" lower="-1.2217" upper="1.9199" />
          <dynamics damping="0.1" />
       </joint>

File: models/urdf/ffw_sg2_rev1_follower/ffw_sg2_follower.urdf (robot description, URDF)
Before this commit: robot ffw_sg2_follower, 42 links, 41 joints
Joints:
- joint arm_l_joint7: limit lower=-1.8201 upper=1.5804 effort=1000 velocity=4.8 -> lower=-1.9199 upper=1.2217 effort=1000 velocity=4.8
- joint arm_r_joint7: limit lower=-1.5804 upper=1.8201 effort=1000 velocity=4.8 -> lower=-1.2217 upper=1.9199 effort=1000 velocity=4.8
